File: Untitled/Untitled.kicad_pcb (KiCad board)
At the start: 2 copper layers, 24 parts, among them J1 Conn_02x04_Counter_Clockwise, J2 Barrel_Jack, J3 Screw_Terminal_01x02, J4 Screw_Terminal_01x02, K1 SANYOU_SRD_Form_C, K2 SANYOU_SRD_Form_C, Q1 BC547, Q2 BC547, U1 L7805, U5 NUCLEO-F410RB

Commit message: finished
Parts:
- added MOTOR1: Conn_01x03, Connector_PinHeader_2.54mm:PinHeader_1x03_P2.54mm_Vertical, F.Cu at (154.5, 46.5)
- added MOTOR2: Conn_01x03, Connector_PinHeader_2.54mm:PinHeader_1x03_P2.54mm_Vertical, F.Cu at (150.2, 46.5)
- added REF**: MountingHole_4.3mm_M4, MountingHole:MountingHole_4.3mm_M4, F.Cu at (57.0, 46.5)
- added REF**: MountingHole_4.3mm_M4, MountingHole:MountingHole_4.3mm_M4, F.Cu at (83.0, 118.2)
- D1, D2: footprint Resistor_THT:R_Axial_DIN0207_L6.3mm_D2.5mm_P10.16mm_Horizontal -> Diode_THT:D_A-405_P10.16mm_Horizontal
- J1: moved to B.Cu
- K1, K2: footprint Relay_THT:Relay_SPST_Finder_32.21-x300 -> Relay_THT:Relay_SPDT_SANYOU_SRD_Series_Form_C
- moved J1 81.5 mm to (129.0, 109.2), turned to 180 degrees
- moved MOIST1 63.4 mm to (132.5, 123.0), turned to -90 degrees
- moved LED1 63.1 mm to (148.3, 123.0), turned to -90 degrees
- moved LDR1 62.1 mm to (154.5, 107.4)
- moved LED2 58.8 mm to (154.5, 119.0)
- moved Q1 55.5 mm to (129.3, 101.6), turned to 180 degrees
- moved LEVEL1 55.1 mm to (142.0, 123.0), turned to -90 degrees
- moved C1 51.2 mm to (126.5, 56.5), turned to -90 degrees
- moved Q2 49.9 mm to (128.8, 82.6), turned to 180 degrees
- moved R1 49.3 mm to (126.0, 98.1), turned to 90 degrees
- moved D1 44.9 mm to (130.0, 87.9), turned to -90 degrees
- moved U1 43.9 mm to (134.8, 60.0)
- moved J2 40.1 mm to (131.5, 53.8), turned to -90 degrees
- moved RGB1 40.0 mm to (154.5, 82.7)
- moved R2 39.5 mm to (125.5, 78.5), turned to 90 degrees
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Connections:
- J1 pad 1: tx -> GND
- J1 pad 2: +3.3V -> tx
- J1 pad 5: rx -> unconnected-(J1-Pin_5-Pad5)
- J1 pad 7: unconnected-(J1-Pin_7-Pad7) -> rx
- J1 pad 8: GND -> +3.3V
- R1 pad 2: MOTOR1 -> PUMP
- R2 pad 2: MOTOR1 -> DC
- U5 pad CN10_33: unconnected-(U5B-PA10-PadCN10_33) -> DC
Routing:
- net +5V: track 0.00 -> 326.4 mm
- net A0: track 0.00 -> 126.8 mm, vias 0 -> 1
- net +3.3V: track 0.00 -> 113.1 mm
- net WATERLEVEL: track 0.00 -> 99.7 mm
- net DC: track 0.00 -> 95.3 mm
- net rx: track 0.00 -> 90.7 mm
- net MOISTURE: track 0.00 -> 87.6 mm
- net tx: track 0.00 -> 84.4 mm
- net PUMP: track 0.00 -> 81.6 mm
- net MOTOR1: track 0.00 -> 78.7 mm
- net MOTOR2: track 0.00 -> 77.5 mm
- net GND: track 0.00 -> 63.4 mm, vias 0 -> 2
- net GLED: track 0.00 -> 61.4 mm
- net DHT: track 0.00 -> 59.7 mm
- net BLED: track 0.00 -> 47.4 mm
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- added copper zone on B.Cu, net GND
- added copper zone on F.Cu, net GND
Other:
- board outline added: 107.2 x 86 mm
- board text added: "Created by Jerick for MAPP @ 2024"
