File: Untitled/Untitled.kicad_sch (KiCad schematic)
At the start: 29 parts, among them J2 Barrel_Jack, K1 ADW11, K2 ADW11, K3 ADW11, M1 Pump 1, M2 Fish Feeder, M4 Pump2, Q1 NMOS, Q2 NMOS, Q3 NMOS, Q4 NMOS, U1 DHT11, U2 Moisture Sensor, U3 Water Level Sensor, U4 STM32F103RBTx, U6 ESP-01v090, U7 AP7384-33V

Commit message: started work on thing
Parts:
- removed C2: 0.33uF, symbol Device:C_Small
- removed C3: 0.1uF, symbol Device:C_Small
- removed D1: Grow Light, symbol Device:LED
- removed D3, D4: D, symbol Device:D
- removed K1, K2, K3: ADW11, Relay_THT:Relay_1P1T_NO_10x24x18.8mm_Panasonic_ADW11xxxxW_THT, symbol Relay:ADW11
- removed M1: Pump 1, symbol Motor:Motor_DC
- removed M2: Fish Feeder, symbol Motor:Motor_DC
- removed M4: Pump2, symbol Motor:Motor_DC
- removed Q1, Q2, Q3, Q4: NMOS, symbol Simulation_SPICE:NMOS
- removed R1: Light sensor, symbol Device:R_Photo
- removed R2, R3, R4, R5, R6: 10k, symbol Device:R_Small
- removed U1: DHT11, Sensor:Aosong_DHT11_5.5x12.0_P2.54mm, symbol Sensor:DHT11
- removed U2: Moisture Sensor, symbol My Lib:Moisture_Sensor
- removed U3: Water Level Sensor, symbol My Lib:Moisture_Sensor
- removed U4: STM32F103RBTx, Package_QFP:LQFP-64_10x10mm_P0.5mm, symbol MCU_ST_STM32F1:STM32F103RBTx
- removed U6: ESP-01v090, symbol ESP8266:ESP-01v090
- removed U7: AP7384-33V, Package_TO_SOT_THT:TO-92_Inline_Wide, symbol Regulator_Linear:AP7384-33V
- added C1, C2: 100nF, Capacitor_THT:C_Axial_L3.8mm_D2.6mm_P7.50mm_Horizontal, symbol Device:C
- added D1: D, Resistor_THT:R_Axial_DIN0207_L6.3mm_D2.5mm_P10.16mm_Horizontal, symbol Device:D
- added DHT1, LEVEL1, MOIST1: Conn_01x03, Connector_PinHeader_2.54mm:PinHeader_1x03_P2.54mm_Vertical, symbol Connector_Generic:Conn_01x03
- added J1: Conn_02x04_Counter_Clockwise, Connector_PinHeader_2.54mm:PinHeader_2x04_P2.54mm_Vertical, symbol Connector_Generic:Conn_02x04_Counter_Clockwise
- added J3, J4: Screw_Terminal_01x02, TerminalBlock_MetzConnect:TerminalBlock_MetzConnect_Type011_RT05502HBWC_1x02_P5.00mm_Horizontal, symbol Connector:Screw_Terminal_01x02
- added K1, K2: SANYOU_SRD_Form_C, Relay_THT:Relay_SPST_Finder_32.21-x300, symbol Relay:SANYOU_SRD_Form_C
- added LDR1, RGB1, ULTRA1: Conn_01x04, Connector_PinHeader_2.54mm:PinHeader_1x04_P2.54mm_Vertical, symbol Connector_Generic:Conn_01x04
- added LED1, LED2: Conn_01x02, Connector_PinHeader_2.54mm:PinHeader_1x02_P2.54mm_Vertical, symbol Connector_Generic:Conn_01x02
- added Q1, Q2: BC547, Package_TO_SOT_THT:TO-92_Inline, symbol Transistor_BJT:BC547
- added R1, R2: 1k, Resistor_THT:R_Axial_DIN0207_L6.3mm_D2.5mm_P10.16mm_Horizontal, symbol Device:R
- added U1: L7805, Package_TO_SOT_SMD:TO-252-2, symbol Regulator_Linear:L7805
- added U5: NUCLEO-F410RB, Library:ST_NUCLEO-F410RB, symbol NUCLEO-F410RB:NUCLEO-F410RB
- D2: footprint (none) -> Resistor_THT:R_Axial_DIN0207_L6.3mm_D2.5mm_P10.16mm_Horizontal
- J2: footprint (none) -> Connector_BarrelJack:BarrelJack_Kycon_KLDX-0202-xC_Horizontal
Connections:
- net DHT: now also DHT1.1 (Pin_1), U5.CN9_3 (D2)
- net GND: now also C1.2, C2.2, DHT1.3 (Pin_3), J1.8 (Pin_8), J3.2 (Pin_2), J4.2 (Pin_2), LDR1.3 (Pin_3), LED1.2 (Pin_2), LED2.2 (Pin_2), LEVEL1.2 (Pin_2), MOIST1.2 (Pin_2), Q1.3 (E), Q2.3 (E), RGB1.4 (Pin_4), U1.2 (GND), U5.CN10_20 (GND_CN10), U5.CN10_9 (GND_CN10), U5.CN5_7 (GND_CN5), U5.CN6_6 (GND_CN6), U5.CN6_7 (GND_CN6), U5.CN7_19 (GND_CN7), U5.CN7_20 (GND_CN7), U5.CN7_22 (GND_CN7), U5.CN7_8 (GND_CN7), ULTRA1.4 (Pin_4)
- net MOISTURE: now also MOIST1.3 (Pin_3), U5.CN7_32 (PA4)
- net MOTOR1: now also R1.2, R2.2, U5.CN10_15 (PA7)
- net MOTOR2: now also U5.CN10_13 (PA6)
- net WATERLEVEL: now also LEVEL1.3 (Pin_3), U5.CN7_34 (PB0)
- net at D2.2 (A): now also K2.2, Q2.1 (C)
- net VCC renamed +5V
- net +5V: now also C2.1, D1.1 (K), DHT1.2 (Pin_2), K1.3, K1.5, K2.3, K2.5, LDR1.4 (Pin_4), LEVEL1.1 (Pin_1), MOIST1.1 (Pin_1), U1.3 (OUT), U5.CN6_5 (+5V_CN6), U5.CN7_18 (+5V_CN7), U5.CN7_6 (E5V), ULTRA1.1 (Pin_1)
- net VDC renamed +12V
- net +12V: now also C1.1, U1.1 (IN)
- new net: Q2.2 (B), R2.1
- new net: J3.1 (Pin_1), K1.1
- new net: D1.2 (A), K1.2, Q1.1 (C)
- new net: Q1.2 (B), R1.1
- new net: J4.1 (Pin_1), K2.1
- new net +3.3V: J1.2 (Pin_2), J1.4 (Pin_4), U5.CN6_4 (+3V3_CN6), U5.CN7_16 (+3V3_CN7)
- new net A0: LDR1.1 (Pin_1), U5.CN7_28 (PA0)
- new net BLED: RGB1.3 (Pin_3), U5.CN10_27 (PB4)
- new net D0: LDR1.2 (Pin_2), U5.CN9_2 (D1)
- new net ECHO: U5.CN10_4 (PC6), ULTRA1.3 (Pin_3)
- new net GLED: RGB1.2 (Pin_2), U5.CN10_31 (PB3)
- new net LED1: LED1.1 (Pin_1), U5.CN10_35 (PA2)
- new net LED2: LED2.1 (Pin_1), U5.CN10_37 (PA3)
- new net PUMP: U5.CN7_30 (PA1)
- new net RLED: RGB1.1 (Pin_1), U5.CN10_24 (PB1)
- new net TRIG: U5.CN10_6 (PC5), ULTRA1.2 (Pin_2)
- new net rx: J1.5 (Pin_5), U5.CN7_1 (PC10)
- new net tx: J1.1 (Pin_1), U5.CN7_2 (PC11)
Other:
- note removed: "9 / 11 / 2001"
- note removed: "Automated plant grower x fish alive keeper"
- note removed: "FISH FEEDER MOTOR"
- note removed: "GROW LIGHT"
- note removed: "POWER"
- note removed: "SENSORS"
- note removed: "STM32 dev board"
- note removed: "WATER PUMPS"
- note removed: "WIFI"

Commit message: finished
Parts:
- added MOTOR1, MOTOR2: Conn_01x03, Connector_PinHeader_2.54mm:PinHeader_1x03_P2.54mm_Vertical, symbol Connector_Generic:Conn_01x03
- D1, D2: footprint Resistor_THT:R_Axial_DIN0207_L6.3mm_D2.5mm_P10.16mm_Horizontal -> Diode_THT:D_A-405_P10.16mm_Horizontal
- K1, K2: footprint Relay_THT:Relay_SPST_Finder_32.21-x300 -> Relay_THT:Relay_SPDT_SANYOU_SRD_Series_Form_C
Connections:
- net +3.3V: now also J1.8 (Pin_8); no longer J1.2 (Pin_2)
- net +5V: now also MOTOR1.2 (Pin_2), MOTOR2.2 (Pin_2)
- net GND: now also J1.1 (Pin_1), MOTOR1.3 (Pin_3), MOTOR2.3 (Pin_3); no longer J1.8 (Pin_8)
- net MOTOR1: now also MOTOR1.1 (Pin_1); no longer R1.2, R2.2
- net MOTOR2: now also MOTOR2.1 (Pin_1)
- net PUMP: now also R1.2
- net rx: now also J1.7 (Pin_7); no longer J1.5 (Pin_5)
- net tx: now also J1.2 (Pin_2); no longer J1.1 (Pin_1)
- net DC: now reaches U5.CN10_33 (PA10)
- net DC: now also R2.2
Other:
- moved on the sheet: J3, R1
