File: Untitled/mcu2.kicad_sch (KiCad schematic)
At the start: 3 parts, among them J9 Keypad, U4 STM32F103RBTx

Commit message: started work on thing
Parts:
- removed DS1: WC1602A, Display:WC1602A, symbol Display_Character:WC1602A
- removed J9: Keypad, symbol Connector:Conn_01x08_Pin
- removed U4: STM32F103RBTx, Package_QFP:LQFP-64_10x10mm_P0.5mm, symbol MCU_ST_STM32F1:STM32F103RBTx
Other:
- note removed: "KEYPAD"
- note removed: "LCD"
- note removed: "STM32 dev board"
